Commit message: 调整了小车参数和虚拟世界的构成并解决了rviz读取模型不显示问题

File: ros2_ws/src/my_robot/urdf/robot.urdf.xacro (robot description, xacro)
@@ -57,7 +57,28 @@
   </joint>
   <link name="front_caster_link">
-    <visual><geometry><sphere radius="${caster_radius}"/></geometry></visual>
-    <collision><geometry><sphere radius="${caster_radius}"/></geometry></collision>
-    <inertial><mass value="0.1"/><inertia ixx="0.0001" ixy="0" ixz="0" iyy="0.0001" iyz="0" izz="0.0001"/></inertial>
+    <visual>
+      <origin xyz="0 0 0" rpy="0 0 0"/>
+      <geometry>
+        <sphere radius="${caster_radius}"/>
+      </geometry>
+      <material name="black"><color rgba="0 0 0 1"/></material>
+    </visual>
+    <visual>
+      <origin xyz="0 0 ${(wheel_radius - caster_radius) / 2}" rpy="0 0 0"/>
+      <geometry>
+        <cylinder radius="0.015" length="${wheel_radius - caster_radius}"/>
+      </geometry>
+      <material name="black"/>
+    </visual>
+    <collision>
+      <origin xyz="0 0 0" rpy="0 0 0"/>
+      <geometry>
+        <sphere radius="${caster_radius}"/>
+      </geometry>
+    </collision>
+    <inertial>
+      <mass value="0.1"/>
+      <inertia ixx="0.0001" ixy="0" ixz="0" iyy="0.0001" iyz="0" izz="0.0001"/>
+    </inertial>
   </link>
   <joint name="rear_caster_joint" type="fixed">
@@ -67,7 +88,28 @@
   </joint>
   <link name="rear_caster_link">
-    <visual><geometry><sphere radius="${caster_radius}"/></geometry></visual>
-    <collision><geometry><sphere radius="${caster_radius}"/></geometry></collision>
-    <inertial><mass value="0.1"/><inertia ixx="0.0001" ixy="0" ixz="0" iyy="0.0001" iyz="0" izz="0.0001"/></inertial>
+    <visual>
+      <origin xyz="0 0 0" rpy="0 0 0"/>
+      <geometry>
+        <sphere radius="${caster_radius}"/>
+      </geometry>
+      <material name="black"/>
+    </visual>
+    <visual>
+      <origin xyz="0 0 ${(wheel_radius - caster_radius) / 2}" rpy="0 0 0"/>
+      <geometry>
+        <cylinder radius="0.015" length="${wheel_radius - caster_radius}"/>
+      </geometry>
+      <material name="black"/>
+    </visual>
+    <collision>
+      <origin xyz="0 0 0" rpy="0 0 0"/>
+      <geometry>
+        <sphere radius="${caster_radius}"/>
+      </geometry>
+    </collision>
+    <inertial>
+      <mass value="0.1"/>
+      <inertia ixx="0.0001" ixy="0" ixz="0" iyy="0.0001" iyz="0" izz="0.0001"/>
+    </inertial>
   </link>
   <joint name="lidar_joint" type="fixed">
@@ -124,5 +166,5 @@
     <sensor type="ray" name="laser">
       <pose>0 0 0 0 0 0</pose>
-      <visualize>false</visualize>
+      <visualize>true</visualize>
       <update_rate>10</update_rate>
       <ray>
